File: LFK1.kicad_pcb (KiCad board)
At the start: 2 copper layers, 304.8 x 99.2 mm, 152 parts, among them J1 AVR-ISP-6, SW1 `~, SW10 9, SW11 0, SW12 -_, SW13 =+, SW14 BKSPC, SW15 DEL, SW16 TAB, SW17 Q, SW18 W, SW19 E, SW2 1, SW20 R, SW21 T, SW22 Y, SW23 U, SW24 I, SW25 O, SW26 P, SW27 [{, SW28 ]}, SW29 \|, SW3 2, SW30 HOME, SW31 CAPS, SW32 A, SW33 S, SW34 D, SW35 F, SW36 G, SW37 H, SW38 J, SW39 K, SW4 3, SW40 L, SW41 ;:, SW42 '", SW43 ENTER, SW44 LSHIFT, SW45 Z, SW46 X, SW47 C, SW48 V, SW49 B, SW5 4, SW50 N, SW51 M, SW52 ,<, SW53 .>, SW54 /?, SW55 RSHIFT, SW56 UP, SW57 LCTRL, SW58 LWIN, SW59 LALT, SW6 5, SW60 SPACE, SW61 RALT, SW62 FN, SW63 LEFT, SW64 DOWN, SW65 RIGHT, SW7 6, SW8 7, SW9 8, U1 ATmega32U4-A, U2 PRTR5V0U2X, Y1 Crystal_GND24_Small

Commit message: routing
Parts:
- U1: value ATmega32U4-A -> ATmega32U4-M; footprint Package_QFP:TQFP-44_10x10mm_P0.8mm -> Package_DFN_QFN:QFN-44-1EP_7x7mm_P0.5mm_EP5.2x5.2mm
- moved R2 2.10 mm to (203.1, 137.2)
- moved U1 0.36 mm to (208.8, 131.6)
- moved C3 0.26 mm to (217.9, 117.3)
Routing:
- net +5V: track 195.6 -> 213.8 mm, vias 6 -> 8
- net GND: track 331.2 -> 319.9 mm
- net row4: track 311.9 -> 315.0 mm
- net col4: track 140.1 -> 143.2 mm
- net row3: track 275.2 -> 278.2 mm
- net col5: track 108.3 -> 111.3 mm
- net col3: track 150.8 -> 153.8 mm
- net row2: track 409.1 -> 412.1 mm
- net col6: track 99.4 -> 102.3 mm
- net col2: track 195.3 -> 198.1 mm
- net row1: track 463.8 -> 466.6 mm
- net D-: track 13.4 -> 16.2 mm
- net row0: track 492.5 -> 495.3 mm
- net MISO: track 31.6 -> 34.4 mm
- net col1: track 222.8 -> 225.5 mm
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