File: LFK1.kicad_pcb (KiCad board)
At the start: 2 copper layers, 304.8 x 99.2 mm, 152 parts, among them J1 AVR-ISP-6, SW1 `~, SW10 9, SW11 0, SW12 -_, SW13 =+, SW14 BKSPC, SW15 DEL, SW16 TAB, SW17 Q, SW18 W, SW19 E, SW2 1, SW20 R, SW21 T, SW22 Y, SW23 U, SW24 I, SW25 O, SW26 P, SW27 [{, SW28 ]}, SW29 \|, SW3 2, SW30 HOME, SW31 CAPS, SW32 A, SW33 S, SW34 D, SW35 F, SW36 G, SW37 H, SW38 J, SW39 K, SW4 3, SW40 L, SW41 ;:, SW42 '", SW43 ENTER, SW44 LSHIFT, SW45 Z, SW46 X, SW47 C, SW48 V, SW49 B, SW5 4, SW50 N, SW51 M, SW52 ,<, SW53 .>, SW54 /?, SW55 RSHIFT, SW56 UP, SW57 LCTRL, SW58 LWIN, SW59 LALT, SW6 5, SW60 SPACE, SW61 RALT, SW62 FN, SW63 LEFT, SW64 DOWN, SW65 RIGHT, SW7 6, SW8 7, SW9 8, U1 ATmega32U4-M, U2 PRTR5V0U2X, Y1 Crystal_GND24_Small

Commit message: v1.1.0
Parts:
- C1, C2, C3, C4, C5, C6, C7, C8: footprint Capacitor_SMD:C_0805_2012Metric_Pad1.18x1.45mm_HandSolder -> Capacitor_SMD:C_0805_2012Metric
- F1: footprint Fuse:Fuse_1206_3216Metric_Pad1.42x1.75mm_HandSolder -> Fuse:Fuse_1206_3216Metric
- FB1: footprint Inductor_SMD:L_0805_2012Metric_Pad1.15x1.40mm_HandSolder -> Inductor_SMD:L_0805_2012Metric
- R1, R2, R3, R4, R5, R6: footprint Resistor_SMD:R_0805_2012Metric_Pad1.20x1.40mm_HandSolder -> Resistor_SMD:R_0805_2012Metric
- USB1: footprint Type-C:HRO-TYPE-C-31-M-12-HandSoldering -> Type-C:HRO-TYPE-C-31-M-12-Assembly
- Y1: footprint Crystal:Crystal_SMD_3225-4Pin_3.2x2.5mm_HandSoldering -> Crystal:Crystal_SMD_3225-4Pin_3.2x2.5mm
- moved C3 6.69 mm to (214.2, 122.9), turned to 0 degrees
- moved C4 3.11 mm to (212.9, 136.9)
- moved C8 2.72 mm to (201.9, 127.8)
- moved C6 1.97 mm to (200.9, 125.5)
- moved C7 1.09 mm to (217.2, 128.8)
- moved R6 0.69 mm to (203.6, 54.7)
Routing:
- net Net-(C3-Pad1): track 16.3 -> 11.0 mm
- net VCC: track 25.4 -> 20.3 mm
- net +5V: track 213.8 -> 210.1 mm
- net col14: track 226.5 -> 222.9 mm
- net col13: track 215.7 -> 212.3 mm
- net GND: track 319.9 -> 316.8 mm, vias 81 -> 79
- net col12: track 193.5 -> 190.5 mm
- net RESET: track 65.4 -> 62.6 mm
- net row1: track 466.6 -> 464.1 mm
- net col0: track 248.6 -> 246.1 mm
- net col1: track 225.5 -> 223.1 mm
- net col2: track 198.1 -> 195.8 mm
- net SCK: track 36.6 -> 34.3 mm
- net MOSI: track 38.6 -> 36.3 mm
- net col3: track 153.8 -> 151.6 mm
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